File: esp8266-cc2530.sch (KiCad schematic (older format))
At the start: 35 parts, among them J1 CC2530_programmingHeader, U1 WeMos_D1_mini, U2 AMS1117-3.3, U3 CC2530Fxxx, U4 RFX2401C, Y1 32.768kHz, Y2 32MHz

Commit message: footprints assigned to all parts
Parts:
- removed Y2: 32MHz, Crystal:Crystal_SMD_SeikoEpson_FA238-4Pin_3.2x2.5mm, symbol Device:Crystal
- C18: value 2.2p -> 2.0p; JLCPCB Basic (none) -> Y; LCSC (none) -> C1800
- J1: footprint (none) -> Connector_PinHeader_2.54mm:PinHeader_2x05_P2.54mm_Vertical_SMD; JLCPCB Basic (none) -> No JLCPCB Assembly; LCSC (none) -> C124391
- L1, L2: footprint (none) -> Inductor_SMD:L_0603_1608Metric; JLCPCB Basic (none) -> No JLCPCB Assembly; LCSC (none) -> C251777
- U3: footprint (none) -> Package_DFN_QFN:QFN-40-1EP_6x6mm_P0.5mm_EP4.6x4.6mm
- U4: footprint (none) -> Package_DFN_QFN:QFN-16-1EP_3x3mm_P0.5mm_EP1.7x1.7mm
- Y1: footprint (none) -> Crystal:Crystal_SMD_3215-2Pin_3.2x1.5mm
Connections:
- net GND: now also U3.41 (GND_EP), U4.17 (GND_EP)
- net VCC: now also U4.14 (VDD), U4.16 (VDD)
- net at U4.10 (ANT): now also R5.1
Other:
- note added: "C18 was 2.2pF in CC2530 \nreference design"
- moved on the sheet: C20
Changed lines of the file:
@@
 F 0 "U4" H 9650 4450 50  0000 L CNN
 F 1 "RFX2401C" H 9150 3900 50  0000 L CNN
-F 2 "" H 9200 3600 50  0001 C CNN
+F 2 "Package_DFN_QFN:QFN-16-1EP_3x3mm_P0.5mm_EP1.7x1.7mm" H 9200 3600 50  0001 C CNN
 F 3 "https://lcsc.com/product-detail/RF-Transceiver-ICs_Skyworks-Solutions_RFX2401C_Skyworks-Solutions-RFX2401C_C19213.html/?href=jlc-SMT" H 9200 3600 50  0001 C CNN
 F 4 "C19213" H 9200 3600 50  0001 C CNN "LCSC"
@@
 P 8300 3050
 F 0 "C18" V 8048 3050 50  0000 C CNN
-F 1 "2.2p" V 8139 3050 50  0000 C CNN
+F 1 "2.0p" V 8139 3050 50  0000 C CNN
 F 2 "Capacitor_SMD:C_0805_2012Metric" H 8338 2900 50  0001 C CNN
 F 3 "~" H 8300 3050 50  0001 C CNN
+F 4 "C1800" V 8300 3050 50  0001 C CNN "LCSC"
+F 5 "Y" H 8300 3050 50  0001 C CNN "JLCPCB Basic"
 	1    8300 3050
 	0    -1   1    0
@@
 F 0 "L2" V 7569 3200 50  0000 C CNN
 F 1 "2n" V 7660 3200 50  0000 C CNN
-F 2 "" H 7750 3200 50  0001 C CNN
-F 3 "~" H 7750 3200 50  0001 C CNN
+F 2 "Inductor_SMD:L_0603_1608Metric" H 7750 3200 50  0001 C CNN
+F 3 "https://lcsc.com/product-detail/HF-Inductors_EMTEK-HSC0603-2N0J-T_C251777.html" H 7750 3200 50  0001 C CNN
+F 4 "No JLCPCB Assembly" H 7750 3200 50  0001 C CNN "JLCPCB Basic"
+F 5 "C251777" H 7750 3200 50  0001 C CNN "LCSC"
 	1    7750 3200
 	0    1    1    0
@@
 F 0 "L1" H 7306 2654 50  0000 R CNN
 F 1 "2n" H 7306 2745 50  0000 R CNN
-F 2 "" H 7350 2700 50  0001 C CNN
-F 3 "~" H 7350 2700 50  0001 C CNN
+F 2 "Inductor_SMD:L_0603_1608Metric" H 7350 2700 50  0001 C CNN
+F 3 "https://lcsc.com/product-detail/HF-Inductors_EMTEK-HSC0603-2N0J-T_C251777.html" H 7350 2700 50  0001 C CNN
+F 4 "No JLCPCB Assembly" H 7350 2700 50  0001 C CNN "JLCPCB Basic"
+F 5 "C251777" H 7350 2700 50  0001 C CNN "LCSC"
 	1    7350 2700
 	-1   0    0    1
@@
 F 0 "U3" H 5700 4300 50  0000 L CNN
 F 1 "CC2530Fxxx" H 4650 3350 50  0000 L CNN
-F 2 "" H 5250 3300 50  0001 C CNN
+F 2 "Package_DFN_QFN:QFN-40-1EP_6x6mm_P0.5mm_EP4.6x4.6mm" H 5250 3300 50  0001 C CNN
 F 3 "https://lcsc.com/product-detail/RF-Transceiver-ICs_Texas-Instruments_CC2530F256RHAR_Texas-Instruments-TI-CC2530F256RHAR_C9120.html/?href=jlc-SMT" H 5250 3300 50  0001 C CNN
 F 4 "C9120" H 5250 3300 50  0001 C CNN "LCSC"
@@
 Connection ~ 6200 3500
 Wire Wire Line
-	9200 2750 9200 2400
-Wire Wire Line
-	9350 2400 9350 2450
-Wire Wire Line
 	9700 3800 9600 3800
 Connection ~ 9000 3800
@@
 $EndComp
 $Comp
-L Device:Crystal Y2
-U 1 1 5EA440B6
-P 8300 4600
-F 0 "Y2" H 8300 4868 50  0000 C CNN
-F 1 "32MHz" H 8300 4777 50  0000 C CNN
-F 2 "Crystal:Crystal_SMD_SeikoEpson_FA238-4Pin_3.2x2.5mm" H 8300 4600 50  0001 C CNN
-F 3 "https://lcsc.com/product-detail/SMD-Crystal-Resonators_Seiko-Epson_X1E000021016300_Seiko-Epson-X1E000021016300_C91742.html/?href=jlc-SMT" H 8300 4600 50  0001 C CNN
-F 4 "C91742" H 8300 4600 50  0001 C CNN "LCSC"
-F 5 "N" H 8300 4600 50  0001 C CNN "JLCPCB Basic"
-	1    8300 4600
-	1    0    0    -1
-$EndComp
-$Comp
 L Device:Crystal Y1
 U 1 1 5EA44653
@@
 F 0 "Y1" V 5754 1531 50  0000 L CNN
 F 1 "32.768kHz" V 5500 1250 50  0000 L CNN
-F 2 "" H 5800 1400 50  0001 C CNN
+F 2 "Crystal:Crystal_SMD_3215-2Pin_3.2x1.5mm" H 5800 1400 50  0001 C CNN
 F 3 "https://lcsc.com/product-detail/SMD-Crystal-Resonators_Seiko-Epson_Q13FC1350000400_Seiko-Epson-Q13FC1350000400_C32346.html/?href=jlc-SMT" H 5800 1400 50  0001 C CNN
 F 4 "C32346" V 5800 1400 50  0001 C CNN "LCSC"
@@
 	8600 3250 8700 3250
 Wire Wire Line
-	8550 3650 8700 3650
-Wire Wire Line
-	8700 3650 8700 3350
+	8550 3650 8650 3650
 $Comp
 L Device:C C20
 U 1 1 5EA73629
-P 9650 2450
-F 0 "C20" V 9398 2450 50  0000 C CNN
-F 1 "1u" V 9489 2450 50  0000 C CNN
-F 2 "Capacitor_SMD:C_0805_2012Metric" H 9688 2300 50  0001 C CNN
-F 3 "https://lcsc.com/product-detail/Multilayer-Ceramic-Capacitors-MLCC-SMD-SMT_SAMSUNG_CL21B105KBFNNNE_1uF-105-10-50V_C28323.html/?href=jlc-SMT" H 9650 2450 50  0001 C CNN
-F 4 "C28323" H 9650 2450 50  0001 C CNN "LCSC"
-F 5 "Y" H 9650 2450 50  0001 C CNN "JLCPCB Basic"
-	1    9650 2450
+P 9650 2400
+F 0 "C20" V 9398 2400 50  0000 C CNN
+F 1 "1u" V 9489 2400 50  0000 C CNN
+F 2 "Capacitor_SMD:C_0805_2012Metric" H 9688 2250 50  0001 C CNN
+F 3 "https://lcsc.com/product-detail/Multilayer-Ceramic-Capacitors-MLCC-SMD-SMT_SAMSUNG_CL21B105KBFNNNE_1uF-105-10-50V_C28323.html/?href=jlc-SMT" H 9650 2400 50  0001 C CNN
+F 4 "C28323" H 9650 2400 50  0001 C CNN "LCSC"
+F 5 "Y" H 9650 2400 50  0001 C CNN "JLCPCB Basic"
+	1    9650 2400
 	0    -1   1    0
 $EndComp
@@
 L power:VCC #PWR0112
 U 1 1 5EA3C514
-P 9250 2400
-F 0 "#PWR0112" H 9250 2250 50  0001 C CNN
-F 1 "VCC" H 9267 2573 50  0000 C CNN
-F 2 "" H 9250 2400 50  0001 C CNN
-F 3 "" H 9250 2400 50  0001 C CNN
-	1    9250 2400
-	1    0    0    -1
-$EndComp
-Wire Wire Line
-	9200 2400 9250 2400
-Connection ~ 9250 2400
-Wire Wire Line
-	9250 2400 9350 2400
-Wire Wire Line
-	9350 2450 9500 2450
-Connection ~ 9350 2450
-Wire Wire Line
-	9350 2450 9350 2750
+P 9300 2400
+F 0 "#PWR0112" H 9300 2250 50  0001 C CNN
+F 1 "VCC" H 9317 2573 50  0000 C CNN
+F 2 "" H 9300 2400 50  0001 C CNN
+F 3 "" H 9300 2400 50  0001 C CNN
+	1    9300 2400
+	1    0    0    -1
+$EndComp
 $Comp
 L power:GND #PWR0113
 U 1 1 5EA7FBBC
-P 9800 2450
-F 0 "#PWR0113" H 9800 2200 50  0001 C CNN
-F 1 "GND" V 9805 2322 50  0000 R CNN
-F 2 "" H 9800 2450 50  0001 C CNN
-F 3 "" H 9800 2450 50  0001 C CNN
-	1    9800 2450
+P 9800 2400
+F 0 "#PWR0113" H 9800 2150 50  0001 C CNN
+F 1 "GND" V 9805 2272 50  0000 R CNN
+F 2 "" H 9800 2400 50  0001 C CNN
+F 3 "" H 9800 2400 50  0001 C CNN
+	1    9800 2400
 	0    -1   -1   0
 $EndComp
@@
 $EndComp
 Wire Wire Line
-	9500 2050 9500 2450
-Connection ~ 9500 2450
-Wire Wire Line
-	9800 2050 9800 2450
-Connection ~ 9800 2450
+	9500 2050 9500 2400
+Connection ~ 9500 2400
+Wire Wire Line
+	9800 2050 9800 2400
+Connection ~ 9800 2400
 Text Notes 8500 950  0    50   ~ 0
 TODO\n* add SMA connector\n* add test points
@@
 	0    1    1    0
 $EndComp
-Wire Wire Line
-	9900 3050 10300 3050
 Text Label 8250 3350 2    50   ~ 0
 P1_1
@@
 F 0 "J1" H 1425 1325 50  0000 C CNN
 F 1 "CC2530_programmingHeader" H 1425 1234 50  0000 C CNN
-F 2 "" H 2100 750 50  0001 C CNN
+F 2 "Connector_PinHeader_2.54mm:PinHeader_2x05_P2.54mm_Vertical_SMD" H 2100 750 50  0001 C CNN
 F 3 "" H 2100 750 50  0001 C CNN
+F 4 "C124391" H 1200 950 50  0001 C CNN "LCSC"
+F 5 "No JLCPCB Assembly" H 1200 950 50  0001 C CNN "JLCPCB Basic"
 	1    1200 950
 	1    0    0    -1
@@
 	6000 4450 6000 4650
 $Comp
-L power:GND #PWR?
+L power:GND #PWR0119
 U 1 1 5ED30DC1
 P 6000 4050
-F 0 "#PWR?" H 6000 3800 50  0001 C CNN
+F 0 "#PWR0119" H 6000 3800 50  0001 C CNN
 F 1 "GND" H 6005 3877 50  0000 C CNN
 F 2 "" H 6000 4050 50  0001 C CNN
@@
 Wire Wire Line
 	6250 3700 6250 4250
+Wire Wire Line
+	4050 2500 3850 2500
+Wire Wire Line
+	3850 2500 3850 2600
+Connection ~ 3850 2600
+Wire Wire Line
+	8700 3350 8650 3350
+Wire Wire Line
+	8650 3350 8650 3650
+Wire Wire Line
+	9800 3800 9700 3800
+Connection ~ 9700 3800
+Wire Wire Line
+	9300 2750 9300 2400
+Connection ~ 9300 2400
+Wire Wire Line
+	9300 2400 9400 2400
+Wire Wire Line
+	9400 2750 9400 2400
+Connection ~ 9400 2400
+Wire Wire Line
+	9400 2400 9500 2400
+Wire Wire Line
+	10000 3050 10300 3050
+Text Notes 8200 2600 0    50   ~ 0
+C18 was 2.2pF in CC2530 \nreference design
 $EndSCHEMATC
